Commit message: fix urdf orientation

File: urdf/robot.urdf (robot description, URDF)
Before this commit: robot riptide2017, 7 links, 6 joints
Links:
- link base_link: geometry visual box size=1.016 0.9144 0.6096
Joints:
- joint base_to_left_wheels: origin xyz=-0.4571 0 0 rpy=0 0 0 -> xyz=0 -0.4571 0 rpy=0 0 0
- joint base_to_right_wheels: origin xyz=0.4571 0 0 rpy=0 0 0 -> xyz=0 0.4571 0 rpy=0 0 0
- joint left_to_left_front: origin xyz=0 0.508 0 rpy=0 0 0 -> xyz=0.508 0 0 rpy=0 0 0
- joint left_to_left_read: origin xyz=0 -0.508 0 rpy=0 0 0 -> xyz=-0.508 0 0 rpy=0 0 0
- joint right_to_right_front: origin xyz=0 0.508 0 rpy=0 0 0 -> xyz=0.508 0 0 rpy=0 0 0
- joint right_to_right_rear: origin xyz=0 -0.508 0 rpy=0 0 0 -> xyz=-0.508 0 0 rpy=0 0 0

Commit message: urdf

File: urdf/robot.urdf (robot description, URDF)
Before this commit: robot riptide2017, 7 links, 6 joints
Links:
- removed link left_front_wheel
- removed link left_rear_wheel
- removed link left_wheels
- removed link right_front_wheel
- removed link right_rear_wheel
- removed link right_wheels
- link base_link: geometry visual box size=1.016 0.9144 0.6096; visual cylinder length=0.0381 radius=0.1524
Joints:
- removed joint base_to_left_wheels
- removed joint base_to_right_wheels
- removed joint left_to_left_front
- removed joint left_to_left_read
- removed joint right_to_right_front
- removed joint right_to_right_rear

Commit message: changes

File: urdf/robot.urdf (robot description, URDF)
Before this commit: robot riptide2017, 1 links, 0 joints
Links:
- added link cam_front; visual sphere radius=0.0762
- link base_link: geometry visual box size=0.9144 0.9906 0.0508; visual cylinder length=0.0381 radius=0.0762
Joints:
- added joint cam_front: type fixed, parent base_link, child cam_front, origin xyz=0.1651 0 0.1778 rpy=-1.57 0 -1.57
